File: bugbeest.kicad_blocks/LV2862 500mA 3.3V Converter.kicad_block/LV2862 500mA 3.3V Converter.kicad_pcb (KiCad board)
At the start: 4 copper layers, 14 parts, among them U1 LV2862YDDC

Commit message: debugged design blocks, added encoder footprint
Parts:
- removed C1: 4.7uF, Capacitor_SMD:C_1206_3216Metric
- removed C2: 0.22uF, Capacitor_SMD:C_0805_2012Metric
- removed C3: 0.1uF, Capacitor_SMD:C_0402_1005Metric
- removed C4: 10uF, Capacitor_SMD:C_0805_2012Metric
- removed JP1: Jumper_2_Small_Open, Jumper:SolderJumper-3_P1.3mm_Bridged2Bar12_RoundedPad1.0x1.5mm_NumberLabels
- removed L1: 15uH, Inductor_SMD:L_1210_3225Metric
- removed R1: 100, Resistor_SMD:R_0402_1005Metric
- removed R2, R3: 100k, Resistor_SMD:R_0402_1005Metric
- removed R4: 33.2K, Resistor_SMD:R_0402_1005Metric
- removed R5: 10k, Resistor_SMD:R_0402_1005Metric
- removed TP1: TestPoint, TestPoint:TestPoint_Pad_D1.5mm
- removed U1: LV2862YDDC, Package_TO_SOT_SMD:SOT-23-6
- added C?: 4.7uF, Capacitor_SMD:C_1206_3216Metric, F.Cu at (-25.5, 45.5)
- added C?: 0.22uF, Capacitor_SMD:C_0805_2012Metric, F.Cu at (-27.7, 46.8)
- added C?: 10uF, Capacitor_SMD:C_0805_2012Metric, F.Cu at (-32.7, 42.6)
- added C?: 0.1uF, Capacitor_SMD:C_0402_1005Metric, F.Cu at (-33.6, 45.3)
- added JP?: Jumper_2_Small_Open, Jumper:SolderJumper-3_P1.3mm_Bridged2Bar12_RoundedPad1.0x1.5mm_NumberLabels, F.Cu at (-25.8, 50.1)
- added L?: 15uH, Inductor_SMD:L_1210_3225Metric, F.Cu at (-30.1, 42.8)
- added R?: 100, Resistor_SMD:R_0402_1005Metric, F.Cu at (-32.5, 50.2)
- added R?: 100k, Resistor_SMD:R_0402_1005Metric, F.Cu at (-30.4, 50.2)
- added R?: 33.2K, Resistor_SMD:R_0402_1005Metric, F.Cu at (-34.9, 46.4)
- added R?: 100k, Resistor_SMD:R_0402_1005Metric, F.Cu at (-28.7, 49.8)
- added R?: 10k, Resistor_SMD:R_0402_1005Metric, F.Cu at (-34.9, 48.4)
- added TP?: TestPoint, TestPoint:TestPoint_Pad_D1.5mm, F.Cu at (-25.1, 41.4)
- added U?: LV2862YDDC, Package_TO_SOT_SMD:SOT-23-6, F.Cu at (-31.9, 48.0)
- moved D1 184.2 mm to (-27.6, 42.8)
