File: bugbeest.kicad_blocks/TCA6408 GPIO Expander.kicad_block/TCA6408 GPIO Expander.kicad_sch (KiCad schematic)
At the start: 5 parts, among them U1 TCA6408ARSVR

Commit message: debugged design blocks, added encoder footprint
Connections:
- net VCCI: now reaches R1.1
- net VCCI: now also C1.1, R2.1, U1.15 (VCCI)
- net VCCP: now reaches C2.1, U1.14 (VCCP)
Other:
- moved on the sheet: C1, C2, R1, R2, U1
